File: Christmas Ornaments/Christmas Ornaments.kicad_sch (KiCad schematic)
At the start: 19 parts, among them U1 ATtiny13A-SS, U2 74HC138

Commit message: git commit -a
Parts:
- added J1, J2: PINHD_1x2_Male, Connector_PinHeader_2.54mm:PinHeader_1x02_P2.54mm_Vertical, symbol PCM_SL_Pin_Headers:PINHD_1x2_Male
- U2: footprint PCM_Package_SO_AKL:SOIC-16_3.9x9.9mm_P1.27mm -> Package_SO:SOIC-16_3.9x9.9mm_P1.27mm
Connections:
- net at U2.1 (A0): now also U1.7 (PB2); no longer U1.6 (PB1)
- net at U2.2 (A1): now also U1.6 (PB1); no longer U1.7 (PB2)
- no-connect marks 0 -> 2
Other:
- company: AvariICe -> AvariCe
